File: wasp1.kicad_sch (KiCad schematic)
At the start: 0 parts

Commit message: Schematics right side
Parts:
- added PinsRightBottomA1, PinsRightBottomB1, PinsRightTopA1, PinsRightTopB1: Conn_02x05_Odd_Even, Connector_PinHeader_2.54mm:PinHeader_2x05_P2.54mm_Vertical, symbol Connector_Generic:Conn_02x05_Odd_Even
- added R1, R10, R11, R12, R13, R14, R2, R3, R4, R5, R6, R7, R8, R9, RThumb1, RThumb2: SW_Push, Button_Switch_Keyboard:SW_Cherry_MX_1.00u_PCB, symbol Switch:SW_Push
- added RD1, RD10, RD11, RD12, RD13, RD14, RD15, RD16, RD2, RD3, RD4, RD5, RD6, RD7, RD8, RD9: DIODE, Diode_THT:D_DO-35_SOD27_P7.62mm_Horizontal, symbol pspice:DIODE
- added RJ45_Right1: 8P8C_Shielded, Connector_RJ:RJ45_Ninigi_GE, symbol Connector:8P8C_Shielded
Connections:
- new net GNDREF: RJ45_Right1.SH
- new net RB1: PinsRightBottomA1.3 (Pin_3), RD1.1 (K)
- new net RB10: PinsRightBottomB1.4 (Pin_4), RD4.1 (K)
- new net RB11: PinsRightBottomB1.6 (Pin_6), RD8.1 (K)
- new net RB12: PinsRightBottomB1.8 (Pin_8), RD12.1 (K)
- new net RB13: PinsRightBottomB1.9 (Pin_9), RD13.1 (K)
- new net RB14: PinsRightBottomB1.10 (Pin_10), RD14.1 (K)
- new net RB2: PinsRightBottomA1.5 (Pin_5), RD5.1 (K)
- new net RB3: PinsRightBottomA1.7 (Pin_7), RD9.1 (K)
- new net RB4: PinsRightBottomA1.4 (Pin_4), RD2.1 (K)
- new net RB5: PinsRightBottomA1.6 (Pin_6), RD6.1 (K)
- new net RB6: PinsRightBottomA1.8 (Pin_8), RD10.1 (K)
- new net RB7: PinsRightBottomB1.3 (Pin_3), RD3.1 (K)
- new net RB8: PinsRightBottomB1.5 (Pin_5), RD7.1 (K)
- new net RB9: PinsRightBottomB1.7 (Pin_7), RD11.1 (K)
- new net RBC1: PinsRightBottomA1.1 (Pin_1), RJ45_Right1.1, RThumb2.1
- new net RBC2: PinsRightBottomA1.2 (Pin_2), RJ45_Right1.2, RThumb1.1
- new net RBC3: PinsRightBottomB1.1 (Pin_1), RJ45_Right1.3
- new net RBC4: PinsRightBottomB1.2 (Pin_2), RJ45_Right1.4
- new net RBT1: RD15.1 (K), RThumb1.2
- new net RBT2: RD16.1 (K), RThumb2.2
- new net RR1: RD1.2 (A), RD2.2 (A), RD3.2 (A), RD4.2 (A), RJ45_Right1.5
- new net RR2: RD5.2 (A), RD6.2 (A), RD7.2 (A), RD8.2 (A), RJ45_Right1.6
- new net RR3: RD10.2 (A), RD11.2 (A), RD12.2 (A), RD9.2 (A), RJ45_Right1.7
- new net RR4: RD13.2 (A), RD14.2 (A), RD15.2 (A), RD16.2 (A), RJ45_Right1.8
- new net RT1: PinsRightTopA1.3 (Pin_3), R1.2
- new net RT10: PinsRightTopB1.4 (Pin_4), R10.2
- new net RT11: PinsRightTopB1.6 (Pin_6), R11.2
- new net RT12: PinsRightTopB1.8 (Pin_8), R12.2
- new net RT13: PinsRightTopB1.9 (Pin_9), R13.2
- new net RT14: PinsRightTopB1.10 (Pin_10), R14.2
- new net RT2: PinsRightTopA1.5 (Pin_5), R2.2
- new net RT3: PinsRightTopA1.7 (Pin_7), R3.2
- new net RT4: PinsRightTopA1.4 (Pin_4), R4.2
- new net RT5: PinsRightTopA1.6 (Pin_6), R5.2
- new net RT6: PinsRightTopA1.8 (Pin_8), R6.2
- new net RT7: PinsRightTopB1.3 (Pin_3), R7.2
- new net RT8: PinsRightTopB1.5 (Pin_5), R8.2
- new net RT9: PinsRightTopB1.7 (Pin_7), R9.2
- new net RTC1: PinsRightTopA1.1 (Pin_1), R1.1, R2.1, R3.1
- new net RTC2: PinsRightTopA1.2 (Pin_2), R4.1, R5.1, R6.1
- new net RTC3: PinsRightTopB1.1 (Pin_1), R13.1, R7.1, R8.1, R9.1
- new net RTC4: PinsRightTopB1.2 (Pin_2), R10.1, R11.1, R12.1, R14.1
- no-connect marks 0 -> 4
