File: wasp1.kicad_sch (KiCad schematic)
At the start: 37 parts

Commit message: Finished schematic?
Parts:
- added BlackPill1: YAAJ_WeAct_BlackPill_Part_Like, wasp:YAAJ_WeAct_BlackPill_2, symbol Blackpill:YAAJ_WeAct_BlackPill_Part_Like
- added L1, L10, L11, L12, L13, L14, L15, L2, L3, L4, L5, L6, L7, L8, L9, LThumb1, LThumb2: SW_Push, Button_Switch_Keyboard:SW_Cherry_MX_1.00u_PCB, symbol Switch:SW_Push
- added PinsLeftBottomA1, PinsLeftBottomB1, PinsLeftTopA1, PinsLeftTopB1: Conn_02x05_Odd_Even, Connector_PinHeader_2.54mm:PinHeader_2x05_P2.54mm_Vertical, symbol Connector_Generic:Conn_02x05_Odd_Even
- added RJ45_Left1: 8P8C_Shielded, Connector_RJ:RJ45_Ninigi_GE, symbol Connector:8P8C_Shielded
Connections:
- net GNDREF: now also RJ45_Left1.SH
- new net BP1: BlackPill1.1 (PB12), RJ45_Left1.8
- new net BP2: BlackPill1.2 (PB13), RJ45_Left1.7
- new net BP3: BlackPill1.3 (PB14), RJ45_Left1.6
- new net BP4: BlackPill1.4 (PB15), RJ45_Left1.5
- new net BP5: BlackPill1.5 (PA8), RJ45_Left1.4
- new net BP6: BlackPill1.6 (PA9), RJ45_Left1.3
- new net BP7: BlackPill1.7 (PA10), RJ45_Left1.2
- new net BP8: BlackPill1.8 (PA11), RJ45_Left1.1
- new net LB1: BlackPill1.29 (PA3), PinsLeftBottomA1.3 (Pin_3)
- new net LB10: BlackPill1.10 (PA15), PinsLeftBottomB1.4 (Pin_4)
- new net LB11: BlackPill1.11 (PB3), PinsLeftBottomB1.6 (Pin_6)
- new net LB12: BlackPill1.12 (PB4), PinsLeftBottomB1.8 (Pin_8)
- new net LB13: BlackPill1.13 (PB5), PinsLeftBottomA1.10 (Pin_10)
- new net LB14: BlackPill1.14 (PB6), PinsLeftBottomB1.9 (Pin_9)
- new net LB15: BlackPill1.15 (PB7), PinsLeftBottomB1.10 (Pin_10)
- new net LB2: BlackPill1.28 (PA2), PinsLeftBottomA1.5 (Pin_5)
- new net LB3: BlackPill1.27 (PA1), PinsLeftBottomA1.7 (Pin_7)
- new net LB4: BlackPill1.26 (PA0), PinsLeftBottomA1.4 (Pin_4)
- new net LB5: BlackPill1.25 (RES), PinsLeftBottomA1.6 (Pin_6)
- new net LB6: BlackPill1.24 (PC15), PinsLeftBottomA1.8 (Pin_8)
- new net LB7: BlackPill1.23 (PC14), PinsLeftBottomB1.3 (Pin_3)
- new net LB8: BlackPill1.22 (PC13), PinsLeftBottomB1.5 (Pin_5)
- new net LB9: BlackPill1.9 (PA12), PinsLeftBottomB1.7 (Pin_7)
- new net LBC1: BlackPill1.35 (PB1), LThumb1.1, LThumb2.1, PinsLeftBottomA1.1 (Pin_1)
- new net LBC2: BlackPill1.34 (PB0), PinsLeftBottomA1.2 (Pin_2)
- new net LBC3: BlackPill1.33 (PA7), PinsLeftBottomB1.1 (Pin_1)
- new net LBC4: BlackPill1.32 (PA6), PinsLeftBottomB1.2 (Pin_2)
- new net LBT1: BlackPill1.31 (PA5), LThumb1.2
- new net LBT2: BlackPill1.30 (PA4), LThumb2.2
- new net LT1: L1.2, PinsLeftTopA1.3 (Pin_3)
- new net LT10: L10.2, PinsLeftTopB1.4 (Pin_4)
- new net LT11: L11.2, PinsLeftTopB1.6 (Pin_6)
- new net LT12: L12.2, PinsLeftTopB1.8 (Pin_8)
- new net LT13: L13.2, PinsLeftTopA1.10 (Pin_10)
- new net LT14: L14.2, PinsLeftTopB1.9 (Pin_9)
- new net LT15: L15.2, PinsLeftTopB1.10 (Pin_10)
- new net LT2: L2.2, PinsLeftTopA1.5 (Pin_5)
- new net LT3: L3.2, PinsLeftTopA1.7 (Pin_7)
- new net LT4: L4.2, PinsLeftTopA1.4 (Pin_4)
- new net LT5: L5.2, PinsLeftTopA1.6 (Pin_6)
- new net LT6: L6.2, PinsLeftTopA1.8 (Pin_8)
- new net LT7: L7.2, PinsLeftTopB1.3 (Pin_3)
- new net LT8: L8.2, PinsLeftTopB1.5 (Pin_5)
- new net LT9: L9.2, PinsLeftTopB1.7 (Pin_7)
- new net LTC1: L1.1, L2.1, L3.1, PinsLeftTopA1.1 (Pin_1)
- new net LTC2: L13.1, L4.1, L5.1, L6.1, PinsLeftTopA1.2 (Pin_2)
- new net LTC3: L14.1, L7.1, L8.1, L9.1, PinsLeftTopB1.1 (Pin_1)
- new net LTC4: L10.1, L11.1, L12.1, L15.1, PinsLeftTopB1.2 (Pin_2)
- no-connect marks 4 -> 17
