File: wasp1.kicad_pcb (KiCad board)
At the start: 2 copper layers, 156.1 x 167.7 mm, 43 parts

Commit message: Schematics WIP
Parts:
- added ?: , , F.Cu at (163.8, 196.2)
- added Z: SW_Cherry_MX_1.00u_PCB, Button_Switch_Keyboard:SW_Cherry_MX_1.00u_PCB, F.Cu at (168.9, 179.6)
Routing:
- net (no net): track 303.5 -> 0.00 mm
Other:
- outline, holes or cut-outs redrawn
- board text added: "Left"
- board text added: "Right"
Changed lines of the file:
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@@
   )
   (net 0 "")
+  (footprint "" (layer "F.Cu")
+    (at 163.83 196.168)
+    (fp_text reference "" (at 0 0) (layer "F.SilkS")
+      (effects (font (size 1.27 1.27) (thickness 0.15)))
+    )
+    (fp_text value "" (at 0 0) (layer "F.SilkS")
+      (effects (font (size 1.27 1.27) (thickness 0.15)))
+    )
+    (pad "" np_thru_hole circle locked (at 0 0 270) (size 4 4) (drill 4) (layers *.Cu *.Mask))
+  )
   (footprint "Connector_PinHeader_2.54mm:PinHeader_2x05_P2.54mm_Vertical" (layer "F.Cu")
     (at 75.73 165.655 180)
@@
   )
   (footprint "Button_Switch_Keyboard:SW_Cherry_MX_1.00u_PCB" (layer "F.Cu")
+    (at 168.91 179.578 -90)
+    (descr "Cherry MX keyswitch, 1.00u, PCB mount, http://cherryamericas.com/wp-content/uploads/2014/12/mx_cat.pdf")
+    (tags "Cherry MX keyswitch 1.00u PCB")
+    (attr through_hole)
+    (fp_text reference "Z" (at -2.54 -2.794 90) (layer "F.SilkS")
+      (effects (font (size 1 1) (thickness 0.15)))
+    )
+    (fp_text value "SW_Cherry_MX_1.00u_PCB" (at -2.54 12.954 90) (layer "F.Fab")
+      (effects (font (size 1 1) (thickness 0.15)))
+    )
+    (fp_text user "${REFERENCE}" (at -2.54 -2.794 90) (layer "F.Fab")
+      (effects (font (size 1 1) (thickness 0.15)))
+    )
+    (fp_line (start -9.525 12.065) (end -9.525 -1.905) (layer "F.SilkS") (width 0.12))
+    (fp_line (start 4.445 -1.905) (end 4.445 12.065) (layer "F.SilkS") (width 0.12))
+    (fp_line (start 4.445 12.065) (end -9.525 12.065) (layer "F.SilkS") (width 0.12))
+    (fp_line (start -9.525 -1.905) (end 4.445 -1.905) (layer "F.SilkS") (width 0.12))
+    (fp_line (start 6.985 14.605) (end -12.065 14.605) (layer "Dwgs.User") (width 0.15))
+    (fp_line (start 6.985 -4.445) (end 6.985 14.605) (layer "Dwgs.User") (width 0.15))
+    (fp_line (start -12.065 -4.445) (end 6.985 -4.445) (layer "Dwgs.User") (width 0.15))
+    (fp_line (start -12.065 14.605) (end -12.065 -4.445) (layer "Dwgs.User") (width 0.15))
+    (fp_line (start 4.06 11.68) (end -9.14 11.68) (layer "F.CrtYd") (width 0.05))
+    (fp_line (start 4.06 -1.52) (end 4.06 11.68) (layer "F.CrtYd") (width 0.05))
+    (fp_line (start -9.14 11.68) (end -9.14 -1.52) (layer "F.CrtYd") (width 0.05))
+    (fp_line (start -9.14 -1.52) (end 4.06 -1.52) (layer "F.CrtYd") (width 0.05))
+    (fp_line (start -8.89 -1.27) (end 3.81 -1.27) (layer "F.Fab") (width 0.1))
+    (fp_line (start 3.81 11.43) (end -8.89 11.43) (layer "F.Fab") (width 0.1))
+    (fp_line (start 3.81 -1.27) (end 3.81 11.43) (layer "F.Fab") (width 0.1))
+    (fp_line (start -8.89 11.43) (end -8.89 -1.27) (layer "F.Fab") (width 0.1))
+    (pad "" np_thru_hole circle locked (at -7.62 5.08 270) (size 1.7 1.7) (drill 1.7) (layers *.Cu *.Mask))
+    (pad "" np_thru_hole circle locked (at -2.54 5.08 270) (size 4 4) (drill 4) (layers *.Cu *.Mask))
+    (pad "" np_thru_hole circle locked (at 2.54 5.08 270) (size 1.7 1.7) (drill 1.7) (layers *.Cu *.Mask))
+    (pad "1" thru_hole circle locked (at 0 0 270) (size 2.2 2.2) (drill 1.5) (layers *.Cu *.Mask))
+    (pad "2" thru_hole circle locked (at -6.35 2.54 270) (size 2.2 2.2) (drill 1.5) (layers *.Cu *.Mask))
+    (model "${KICAD6_3DMODEL_DIR}/Button_Switch_Keyboard.3dshapes/SW_Cherry_MX_1.00u_PCB.wrl"
+      (offset (xyz 0 0 0))
+      (scale (xyz 1 1 1))
+      (rotate (xyz 0 0 0))
+    )
+  )
+  (footprint "Button_Switch_Keyboard:SW_Cherry_MX_1.00u_PCB" (layer "F.Cu")
     (at 149.8 154.03 -90)
     (descr "Cherry MX keyswitch, 1.00u, PCB mount, http://cherryamericas.com/wp-content/uploads/2014/12/mx_cat.pdf")
@@
   )
   (footprint "Button_Switch_Keyboard:SW_Cherry_MX_1.00u_PCB" (layer "F.Cu")
-    (at 48.26 121.702102 135)
+    (at 48.26 121.7021 135)
     (descr "Cherry MX keyswitch, 1.00u, PCB mount, http://cherryamericas.com/wp-content/uploads/2014/12/mx_cat.pdf")
     (tags "Cherry MX keyswitch 1.00u PCB")
@@
   )
   (footprint "Button_Switch_Keyboard:SW_Cherry_MX_1.00u_PCB" (layer "F.Cu")
-    (at 33.655 107.097102 135)
+    (at 33.655 107.0971 135)
     (descr "Cherry MX keyswitch, 1.00u, PCB mount, http://cherryamericas.com/wp-content/uploads/2014/12/mx_cat.pdf")
     (tags "Cherry MX keyswitch 1.00u PCB")
@@
   )
   (footprint "Button_Switch_Keyboard:SW_Cherry_MX_1.00u_PCB" (layer "B.Cu")
-    (at 153.778949 108.893154 -45)
+    (at 153.7789 108.8932 -45)
     (descr "Cherry MX keyswitch, 1.00u, PCB mount, http://cherryamericas.com/wp-content/uploads/2014/12/mx_cat.pdf")
     (tags "Cherry MX keyswitch 1.00u PCB")
@@
   )
   (footprint "Button_Switch_Keyboard:SW_Cherry_MX_1.00u_PCB" (layer "B.Cu")
-    (at 139.173949 94.288154 -45)
+    (at 139.1739 94.2882 -45)
     (descr "Cherry MX keyswitch, 1.00u, PCB mount, http://cherryamericas.com/wp-content/uploads/2014/12/mx_cat.pdf")
     (tags "Cherry MX keyswitch 1.00u PCB")
@@
   )
   (gr_line (start 19.39 88.705) (end 19.625 20.84) (layer "Edge.Cuts") (width 0.1))
-  (gr_line (start 126.775 88.705) (end 126.775 61.48) (layer "Edge.Cuts") (width 0.1))
+  (gr_line (start 126.775 88.659872) (end 126.775 61.48) (layer "Edge.Cuts") (width 0.1))
   (gr_line (start 26.67 88.705) (end 26.67 90.805) (layer "Edge.Cuts") (width 0.1))
   (gr_line (start 70.885 188.515) (end 70.885 150.495) (layer "Edge.Cuts") (width 0.1))
@@
   (gr_line (start 68.11 188.515) (end 19.85 188.515) (layer "Edge.Cuts") (width 0.1))
   (gr_line (start 126.775 20.84) (end 175.035 20.84) (layer "Edge.Cuts") (width 0.1))
-  (gr_line (start 175.2 118.504872) (end 156.15 118.504872) (layer "Edge.Cuts") (width 0.1))
+  (gr_line (start 175.035 118.504872) (end 156.15 118.504872) (layer "Edge.Cuts") (width 0.1))
   (gr_line (start 175.035 118.504872) (end 175.035 20.84) (layer "Edge.Cuts") (width 0.1))
   (gr_line (start 67.945 150.495) (end 68.11 188.515) (layer "Edge.Cuts") (width 0.1))
@@
   (gr_line (start 126.775 57.785) (end 126.775 20.84) (layer "Edge.Cuts") (width 0.1))
   (gr_line (start 124 88.705) (end 32.385 88.705) (layer "Edge.Cuts") (width 0.1))
+  (gr_text "Right" (at 154.94 62.23 -90) (layer "B.SilkS")
+    (effects (font (size 10 10) (thickness 0.15)) (justify mirror))
+  )
+  (gr_text "Left" (at 31.75 127) (layer "F.SilkS")
+    (effects (font (size 5 5) (thickness 0.15)))
+  )
   (gr_text "PinHeader_2x05_P2.54mm_Horizontal" (at 85.157 46.931 -90) (layer "B.Fab")
     (effects (font (size 1 1) (thickness 0.15)) (justify mirror))
@@
     (effects (font (size 1 1) (thickness 0.15)))
   )
-  (segment (start 26.035 61.595) (end 26.035 72.724) (width 0.25) (layer "F.Cu") (net 0))
-  (segment (start 29.21 20.955) (end 119.38 20.955) (width 0.2) (layer "F.Cu") (net 0))
-  (segment (start 26.095 26.73) (end 24.765 25.4) (width 0.2) (layer "F.Cu") (net 0))
-  (segment (start 28.635 24.705) (end 31.115 22.225) (width 0.2) (layer "F.Cu") (net 0))
-  (segment (start 121.695 23.27) (end 121.695 43.7) (width 0.2) (layer "F.Cu") (net 0))
-  (segment (start 31.115 22.225) (end 118.745 22.225) (width 0.2) (layer "F.Cu") (net 0))
-  (segment (start 118.745 22.225) (end 119.155 22.635) (width 0.2) (layer "F.Cu") (net 0))
-  (segment (start 119.155 22.635) (end 119.155 43.7) (width 0.2) (layer "F.Cu") (net 0))
-  (segment (start 28.575 34.925) (end 28.575 47.244) (width 0.2) (layer "F.Cu") (net 0))
-  (segment (start 26.035 60.325) (end 26.035 61.595) (width 0.2) (layer "F.Cu") (net 0))
-  (segment (start 26.095 41.275) (end 26.095 60.265) (width 0.2) (layer "F.Cu") (net 0))
-  (segment (start 26.095 60.265) (end 26.035 60.325) (width 0.2) (layer "F.Cu") (net 0))
-  (segment (start 26.095 41.275) (end 26.095 26.73) (width 0.2) (layer "F.Cu") (net 0))
-  (segment (start 119.38 20.955) (end 121.695 23.27) (width 0.2) (layer "F.Cu") (net 0))
-  (segment (start 28.635 34.925) (end 28.635 34.865) (width 0.2) (layer "F.Cu") (net 0))
-  (segment (start 24.765 25.4) (end 29.21 20.955) (width 0.2) (layer "F.Cu") (net 0))
-  (segment (start 28.635 34.865) (end 28.635 24.705) (width 0.2) (layer "F.Cu") (net 0))
-  (segment (start 28.635 34.865) (end 28.575 34.925) (width 0.2) (layer "F.Cu") (net 0))
 )

Commit message: Schematics right side
Parts:
- removed ?: , 
- removed A, B, BackSpace, C, Comma, D, Dot, E, Enter, F, G, H, I, J, K, L, M, N, O, P, Q, R, S, Space, T, Tab, U, V, W, X, Y, Z (x2): SW_Cherry_MX_1.00u_PCB, Button_Switch_Keyboard:SW_Cherry_MX_1.00u_PCB
- removed BlackPill: WeAct BlackPill, BlackPill:YAAJ_WeAct_BlackPill_SWD_2
- removed PinHeaderLeftBottomA, PinHeaderLeftBottomB, PinHeaderLeftTopA, PinHeaderLeftTopB, PinHeaderRightBottomA, PinHeaderRightBottomB, PinHeaderRightTopA, PinHeaderRightTopB: PinHeader_2x05_P2.54mm_Vertical, Connector_PinHeader_2.54mm:PinHeader_2x05_P2.54mm_Vertical
- removed RJ45Left, RJ45Right: RJ45_Ninigi_GE, Connector_RJ:RJ45_Ninigi_GE
- added PinsRightBottomA1: Conn_02x05_Odd_Even, Connector_PinHeader_2.54mm:PinHeader_2x05_P2.54mm_Vertical, F.Cu at (129.4, 33.7)
- added PinsRightBottomB1: Conn_02x05_Odd_Even, Connector_PinHeader_2.54mm:PinHeader_2x05_P2.54mm_Vertical, F.Cu at (129.4, 71.5)
- added PinsRightTopA1: Conn_02x05_Odd_Even, Connector_PinHeader_2.54mm:PinHeader_2x05_P2.54mm_Vertical, F.Cu at (119.0, 33.7)
- added PinsRightTopB1: Conn_02x05_Odd_Even, Connector_PinHeader_2.54mm:PinHeader_2x05_P2.54mm_Vertical, F.Cu at (119.0, 71.0)
- added R1: SW_Push, Button_Switch_Keyboard:SW_Cherry_MX_1.00u_PCB, F.Cu at (109.2, 33.9)
- added R10: SW_Push, Button_Switch_Keyboard:SW_Cherry_MX_1.00u_PCB, F.Cu at (50.3, 30.9)
- added R11: SW_Push, Button_Switch_Keyboard:SW_Cherry_MX_1.00u_PCB, F.Cu at (50.3, 50.7)
- added R12: SW_Push, Button_Switch_Keyboard:SW_Cherry_MX_1.00u_PCB, F.Cu at (50.3, 70.0)
- added R13: SW_Push, Button_Switch_Keyboard:SW_Cherry_MX_1.00u_PCB, F.Cu at (30.6, 43.7)
- added R14: SW_Push, Button_Switch_Keyboard:SW_Cherry_MX_1.00u_PCB, F.Cu at (30.9, 63.4)
- added R2: SW_Push, Button_Switch_Keyboard:SW_Cherry_MX_1.00u_PCB, F.Cu at (109.0, 53.6)
- added R3: SW_Push, Button_Switch_Keyboard:SW_Cherry_MX_1.00u_PCB, F.Cu at (109.2, 73.2)
- added R4: SW_Push, Button_Switch_Keyboard:SW_Cherry_MX_1.00u_PCB, F.Cu at (89.5, 31.9)
- added R5: SW_Push, Button_Switch_Keyboard:SW_Cherry_MX_1.00u_PCB, F.Cu at (89.7, 51.6)
- added R6: SW_Push, Button_Switch_Keyboard:SW_Cherry_MX_1.00u_PCB, F.Cu at (89.7, 71.0)
- added R7: SW_Push, Button_Switch_Keyboard:SW_Cherry_MX_1.00u_PCB, F.Cu at (69.8, 25.9)
- added R8: SW_Push, Button_Switch_Keyboard:SW_Cherry_MX_1.00u_PCB, F.Cu at (70.2, 45.3)
- added R9: SW_Push, Button_Switch_Keyboard:SW_Cherry_MX_1.00u_PCB, F.Cu at (69.7, 65.2)
- added RD1: DIODE, Diode_THT:D_DO-35_SOD27_P7.62mm_Horizontal, F.Cu at (160.8, 62.5)
- added RD10: DIODE, Diode_THT:D_DO-35_SOD27_P7.62mm_Horizontal, F.Cu at (169.3, 51.3)
- added RD11: DIODE, Diode_THT:D_DO-35_SOD27_P7.62mm_Horizontal, F.Cu at (149.7, 62.6)
- added RD12: DIODE, Diode_THT:D_DO-35_SOD27_P7.62mm_Horizontal, F.Cu at (147.2, 51.3)
- added RD13: DIODE, Diode_THT:D_DO-35_SOD27_P7.62mm_Horizontal, F.Cu at (146.2, 62.6)
- added RD14: DIODE, Diode_THT:D_DO-35_SOD27_P7.62mm_Horizontal, F.Cu at (149.8, 73.4)
- added RD15: DIODE, Diode_THT:D_DO-35_SOD27_P7.62mm_Horizontal, F.Cu at (160.8, 85.2)
- added RD16: DIODE, Diode_THT:D_DO-35_SOD27_P7.62mm_Horizontal, F.Cu at (153.5, 73.4)
- added RD2: DIODE, Diode_THT:D_DO-35_SOD27_P7.62mm_Horizontal, F.Cu at (161.9, 51.3)
- added RD3: DIODE, Diode_THT:D_DO-35_SOD27_P7.62mm_Horizontal, F.Cu at (160.8, 73.4)
- added RD4: DIODE, Diode_THT:D_DO-35_SOD27_P7.62mm_Horizontal, F.Cu at (153.3, 62.6)
- added RD5: DIODE, Diode_THT:D_DO-35_SOD27_P7.62mm_Horizontal, F.Cu at (139.8, 51.3)
- added RD6: DIODE, Diode_THT:D_DO-35_SOD27_P7.62mm_Horizontal, F.Cu at (154.6, 51.3)
- added RD7: DIODE, Diode_THT:D_DO-35_SOD27_P7.62mm_Horizontal, F.Cu at (157.2, 73.4)
- added RD8: DIODE, Diode_THT:D_DO-35_SOD27_P7.62mm_Horizontal, F.Cu at (146.2, 73.4)
- added RD9: DIODE, Diode_THT:D_DO-35_SOD27_P7.62mm_Horizontal, F.Cu at (156.8, 62.7)
- added RJ45_Right1: 8P8C_Shielded, Connector_RJ:RJ45_Ninigi_GE, F.Cu at (141.6, 26.1)
- added RThumb1: SW_Push, Button_Switch_Keyboard:SW_Cherry_MX_1.00u_PCB, B.Cu at (161.4, 105.7)
- added RThumb2: SW_Push, Button_Switch_Keyboard:SW_Cherry_MX_1.00u_PCB, B.Cu at (147.4, 91.8)
Other:
- outline, holes or cut-outs redrawn
- board text removed: "PinHeader_2x05_P2.54mm_Horizontal"

Commit message: Finished schematic?
Parts:
- added BlackPill1: YAAJ_WeAct_BlackPill_Part_Like, wasp:YAAJ_WeAct_BlackPill_2, F.Cu at (39.9, 185.8)
